File: src/little-bird.kicad_pcb (KiCad board)
At the start: 2 copper layers, 51.7 x 99 mm, 13 parts, among them Q1 PNP

Commit message: Update PCB
Parts:
- added R5: R, Resistor_THT:R_Axial_DIN0207_L6.3mm_D2.5mm_P7.62mm_Horizontal, F.Cu at (157.0, 104.6)
- Q1: value PNP -> NPN
- moved Q1 0.37 mm to (161.4, 78.3)
Connections:
- C1 pad 1: Net-(BT1-+) -> Net-(D1-A)
- Q1 pad 3: Net-(D1-A) -> Net-(Q1-E)
- R4 pad 1: Net-(R4-Pad1) -> Net-(Q1-B)
- R4 pad 2: Net-(Q1-B) -> Net-(BT1--)
- RV1 pad 1: unconnected-(RV1-Pad1) -> Net-(Q1-E)
- RV1 pad 2: Net-(R4-Pad1) -> Net-(D1-A)
- RV1 pad 3: Net-(BT1-+) -> unconnected-(RV1-Pad3)
Routing:
- net Net-(Q1-B): track 8.54 -> 43.2 mm
- net Net-(Q1-E): track 0.00 -> 26.5 mm
- net Net-(BT1-+): track 76.9 -> 58.1 mm, vias 0 -> 1
- net Net-(R4-Pad1): track 14.0 -> 0.00 mm
- net Net-(D1-A): track 148.2 -> 145.3 mm
- net Net-(D3-K): track 12.7 -> 13.6 mm
- net Net-(BT1--): track 103.3 -> 104.0 mm
