File: src/little-bird.kicad_sch (KiCad schematic)
At the start: 11 parts, among them Q1 PNP

Commit message: Update PCB
Parts:
- removed Q1: PNP, Package_TO_SOT_THT:TO-92L_HandSolder, symbol Simulation_SPICE:PNP
- added Q1: NPN, Package_TO_SOT_THT:TO-92L_HandSolder, symbol Simulation_SPICE:NPN
- added R5: R, Resistor_THT:R_Axial_DIN0207_L6.3mm_D2.5mm_P7.62mm_Horizontal, symbol Device:R
Connections:
- net at BT1.2 (-), C1.2, R1.2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: now also R4.2
- net at D1.2 (A), D2.2 (A), D3.2 (A): now also C1.1, RV1.2
- net at R4.1: now also Q1.2 (B), R5.1; no longer RV1.2
- net at RV1.1: now also Q1.3 (E)
- new net: BT1.1 (+), Q1.1 (C), R5.2
- now unconnected: RV1.3
Other:
- moved on the sheet: C1, R4, RV1
